Commit message: Small fix human bio model

File: urdf/human_bio.urdf (robot description, URDF)
Before this commit: robot human_model, 53 links, 52 joints
Joints:
- joint TorsoTrans: limit lower=-30 upper=30 effort=15 velocity=5 -> lower=-1 upper=1 effort=15 velocity=5
- joint lShoulderTransX: limit lower=-30 upper=30 effort=15 velocity=5 -> lower=-1 upper=1 effort=15 velocity=5
- joint lShoulderTransY: limit lower=-30 upper=30 effort=15 velocity=5 -> lower=-1 upper=1 effort=15 velocity=5
- joint lShoulderTransZ: limit lower=-30 upper=30 effort=15 velocity=5 -> lower=-1 upper=1 effort=15 velocity=5
- joint rElbowY: limit lower=-3.15 upper=3.15 effort=15 velocity=5 -> lower=-.5 upper=.5 effort=15 velocity=5
- joint rShoulderTransX: limit lower=-30 upper=30 effort=15 velocity=5 -> lower=-1 upper=1 effort=15 velocity=5
- joint rShoulderTransY: limit lower=-30 upper=30 effort=15 velocity=5 -> lower=-1 upper=1 effort=15 velocity=5
- joint rShoulderTransZ: limit lower=-30 upper=30 effort=15 velocity=5 -> lower=-1 upper=1 effort=15 velocity=5

Commit message: Add a default configuration and resize the geometry for better looks

File: urdf/human_bio.urdf (robot description, URDF)
Before this commit: robot human_model, 53 links, 52 joints
Links:
- link lFemur: geometry visual cylinder length=0.45 radius=0.0871
- link lFoot: geometry visual box size=0.25 0.1488 0.063
- link lHand: geometry visual box size=0.07 0.10 .025
- link lHumerus: geometry visual cylinder length=0.2475 radius=0.045
- link lRadius: geometry visual cylinder length=0.281 radius=0.04
- link rFemur: geometry visual cylinder length=0.45 radius=0.0871
- link rFoot: geometry visual box size=0.25 0.1488 0.063
- link rHand: geometry visual box size=0.07 0.10 .025
- link rHumerus: geometry visual cylinder length=0.2475 radius=0.045
- link rRadius: geometry visual cylinder length=0.281 radius=0.04
Joints:
- joint lAnkleZ: origin xyz=0 0 0 -> xyz=0.07 0 0
- joint rAnkleZ: origin xyz=0 0 0 -> xyz=0.07 0 0

Commit message: Fix most discrepencies with other models

File: urdf/human_bio.urdf (robot description, URDF)
Before this commit: robot human_model, 53 links, 52 joints
Links:
- link PelvisBody: geometry visual cylinder length=0.22 radius=0.14
- link rHumerus: geometry visual cylinder length=0.3475 radius=0.053
- link rRadius: geometry visual cylinder length=0.31 radius=0.04
Joints:
- joint TorsoY: axis 0 1 0 -> 0 0 1
- joint TorsoZ: axis 0 0 1 -> 0 1 0
- joint rShoulderTransY: axis 0 1 0 -> 0 0 1
- joint rShoulderTransZ: axis 0 0 1 -> 0 -1 0
- joint rShoulderY1: origin xyz=0 0 0 -> xyz=0 0 0 rpy=1.570796326 0 0
- joint rWristX: limit lower=-3.14 upper=0 effort=15 velocity=5 -> lower=-3.14 upper=3.15 effort=15 velocity=5

Commit message: Fix other issues with the kenamtics

File: urdf/human_bio.urdf (robot description, URDF)
Before this commit: robot human_model, 53 links, 52 joints
Joints:
- joint PelvisRotZ: origin xyz=0.037432 0 0.139749 -> xyz=0 0 0
- joint TorsoZ: axis 0 1 0 -> 0 -1 0

Commit message: Add semantic descriptor

File: urdf/human_bio.urdf (robot description, URDF)
Before this commit: robot human_model, 53 links, 52 joints
Joints:
- joint TorsoTrans: limit lower=-1 upper=1 effort=15 velocity=5 -> (none); type prismatic -> fixed
- joint lShoulderX: origin xyz=-0.048632 0.23982 0.288822 -> xyz=-0.048632 0.23982 0.288822 rpy=-1.570796326 0 0
